File: Circuito/robotsito pcb.kicad_pcb (KiCad board)
At the start: 2 copper layers, 50 x 50 mm, 5 parts, among them J1 Screw_Terminal_01x04, P1 Conn_DRV8833_1, P2 Conn_DRV8833_2

Commit message: PCB v1.1
Parts:
- added C1: C, Capacitor_THT:C_Disc_D6.0mm_W2.5mm_P5.00mm, F.Cu at (205.5, 64.6)
- added C2: C, Capacitor_THT:C_Disc_D6.0mm_W2.5mm_P5.00mm, F.Cu at (213.0, 64.6)
- moved Conn_DRV8833_Entrada1 18.6 mm to (189.2, 89.4), turned to 180 degrees
- moved P1 7.29 mm to (205.8, 90.7)
- moved P2 7.29 mm to (205.4, 72.4)
- moved J1 4.68 mm to (207.9, 57.5)
Connections:
- Conn_DRV8833_Entrada1 pad 1: /AIN1 -> /AIN2
- Conn_DRV8833_Entrada1 pad 2: /AIN2 -> /AIN1
- J1 pad 1: /BO2 -> /BO1
- J1 pad 2: /BO1 -> /BO2
Routing:
- net /BIN2: track 0.00 -> 33.6 mm
- net /BIN1: track 0.00 -> 30.0 mm
- net /AIN1: track 0.00 -> 23.2 mm
- net /AIN2: track 0.00 -> 21.8 mm
- net /AO1: track 0.00 -> 16.9 mm
- net /BO1: track 0.00 -> 16.9 mm
- net /BO2: track 0.00 -> 14.9 mm
- net /AO2: track 0.00 -> 14.9 mm
