File: Circuito/robotsito pcb.kicad_sch (KiCad schematic)
At the start: 5 parts, among them J1 Screw_Terminal_01x04, P1 Conn_DRV8833_1, P2 Conn_DRV8833_2

Commit message: PCB v1.1
Parts:
- added C1, C2: C, Capacitor_THT:C_Disc_D6.0mm_W2.5mm_P5.00mm, symbol Device:C
- Batería1: renamed from Batería; footprint (none) -> TerminalBlock:TerminalBlock_Altech_AK300-2_P5.00mm
- J1: footprint (none) -> Connector_PinHeader_2.54mm:PinHeader_1x04_P2.54mm_Vertical
- P1, P2: footprint (none) -> Connector_PinHeader_2.54mm:PinHeader_1x08_P2.54mm_Vertical
- renumbered Conn_DRV8833_Entrada to Conn_DRV8833_Entrada1
Connections:
- net AIN1: now also Conn_DRV8833_Entrada1.2 (Pin_2); no longer Conn_DRV8833_Entrada1.1 (Pin_1)
- net AIN2: now also Conn_DRV8833_Entrada1.1 (Pin_1); no longer Conn_DRV8833_Entrada1.2 (Pin_2)
- net AO1: now also C2.2
- net AO2: now also C2.1
- net BO1: now also J1.1 (Pin_1), C1.1; no longer J1.2 (Pin_2)
- net BO2: now also J1.2 (Pin_2), C1.2; no longer J1.1 (Pin_1)
Other:
- moved on the sheet: J1
